File: hw/v0p9p5/ras_pi_supercap_ups.kicad_pcb (KiCad board)
At the start: 2 copper layers, 65 x 56 mm, 67 parts, among them J1 Raspberry_Pi_2_3, J10 Conn_01x03, J12 171826-4, J2 Raspberry_Pi_2_3, J3 Conn_01x05, J4 Conn_01x03, J6 Conn_01x04, J7 Conn_01x03, J8 Conn_02x03_Odd_Even, J9 LEDs and Buttons, Q1 IRF5305, U1 KA431SMFTF, U2 KA431SMFTF, U3 KA431SMFTF, U4 KA431SMFTF, U5 KA431SMFTF, U6 LM2596S-5, U7 L7805, U8 ATtiny85-20P, U9 STC8H1K08

Commit message: updates... pulled in buck conv
Parts:
- removed the J2 at (58.3, 112.4)
- removed the J6 at (53.5, 132.4)
- removed JP2, JP3: SolderJumper_2_Open, Jumper:SolderJumper-2_P1.3mm_Open_RoundedPad1.0x1.5mm
- removed REF**: OSHW-Symbol_6.7x6mm_SilkScreen, Symbol:OSHW-Symbol_6.7x6mm_SilkScreen
- removed REF**: KiCad-Logo2_5mm_SilkScreen, Symbol:KiCad-Logo2_5mm_SilkScreen
- removed TP1: TestPoint_Small, TestPoint:TestPoint_THTPad_D1.0mm_Drill0.5mm
- removed the U6 at (90.4, 123.1)
- removed the U7 at (71.6, 126.1)
- added C13: 10u, Capacitor_SMD:C_0805_2012Metric, F.Cu at (61.4, 109.8)
- added C14: 100n, Capacitor_SMD:C_0805_2012Metric, F.Cu at (61.4, 107.8)
- added C15: 4.7u, Capacitor_SMD:C_0805_2012Metric, F.Cu at (101.8, 118.1)
- added C16: 4.7u, Capacitor_SMD:C_0805_2012Metric, F.Cu at (99.8, 118.1)
- added C17: 4.7n, Capacitor_SMD:C_0805_2012Metric, F.Cu at (97.8, 118.2)
- added C18: 100n, Capacitor_SMD:C_0805_2012Metric, F.Cu at (93.3, 115.8)
- added C19: 10n, Capacitor_SMD:C_0805_2012Metric, F.Cu at (101.9, 114.7)
- added C20: 4.7n, Capacitor_SMD:C_0805_2012Metric, F.Cu at (85.9, 113.6)
- added C21: 33u, Capacitor_SMD:C_0805_2012Metric, F.Cu at (76.3, 117.1)
- added C22: 39p, Capacitor_SMD:C_0805_2012Metric, F.Cu at (85.9, 117.0)
- added C23: 33u, Capacitor_SMD:C_0805_2012Metric, F.Cu at (79.6, 117.0)
- added D5: Green, LED_SMD:LED_0805_2012Metric, F.Cu at (113.0, 134.7)
- added D8: B340A, Diode_SMD:D_SMA, F.Cu at (83.6, 110.0)
- added J9: Test Points, Connector_PinHeader_1.00mm:PinHeader_1x03_P1.00mm_Vertical, F.Cu at (70.8, 116.3)
- added L1: 6.8uH, raspberrypi_supercap_ups_lib:Sunltech_SLO0530H, F.Cu at (77.0, 111.6)
- added R12: 10k, Resistor_SMD:R_0805_2012Metric, F.Cu at (76.6, 121.3)
- added R13: 2.2k, Resistor_SMD:R_0805_2012Metric, F.Cu at (80.0, 121.3)
- added R14: 1k, Resistor_SMD:R_0805_2012Metric, F.Cu at (92.2, 131.7)
- added R22: 68.1k, Resistor_SMD:R_0805_2012Metric, F.Cu at (99.9, 114.7)
- added R23: 49.9k, Resistor_SMD:R_0805_2012Metric, F.Cu at (83.8, 113.6)
- added R24: 0, Resistor_SMD:R_0805_2012Metric, F.Cu at (88.0, 117.1)
- added R25: 10.2k, Resistor_SMD:R_0805_2012Metric, F.Cu at (83.3, 116.3)
- added R26: 2k, Resistor_SMD:R_0805_2012Metric, F.Cu at (83.3, 118.4)
- added SW1: Reset, Button_Switch_THT:SW_PUSH_6mm_H4.3mm, F.Cu at (113.4, 112.6)
- added U8: TPS54331DR, raspberrypi_supercap_ups_lib:SOIC127P599X175-8N, F.Cu at (93.5, 112.0)
- C10, C7, C8: value 22u 10V X7R -> 10u
- C11: value 22u 10V X7R -> 1u
- C12: value 0.1u -> 1u
- C9: value 22u 10V X7R -> 100n
- J4: renamed from J8; value Conn_02x03_Odd_Even -> Force Power On; footprint Connector_PinHeader_2.54mm:PinHeader_2x03_P2.54mm_Vertical -> Connector_PinHeader_2.54mm:PinHeader_1x02_P2.54mm_Vertical
- J7: value Conn_01x03 -> STLinkV2 Connector; footprint Connector_PinHeader_2.54mm:PinHeader_1x03_P2.54mm_Vertical -> Connector_PinHeader_2.54mm:PinHeader_1x04_P2.54mm_Vertical
- JP1: value SolderJumper_2_Open -> Charge Enb; footprint Jumper:SolderJumper-2_P1.3mm_Open_RoundedPad1.0x1.5mm -> Jumper:SolderJumper-2_P1.3mm_Bridged_RoundedPad1.0x1.5mm; moved to F.Cu
- R20: value 47k -> 10k
- R21: value 47k -> 332k
- U6: renamed from U8; value ATtiny85-20P -> AMS1117-3.3; footprint Package_DIP:DIP-8_W7.62mm -> Package_TO_SOT_SMD:SOT-223-3_TabPin2
- U7: renamed from U9; value STC8H1K08 -> STM8S003F3P
- moved R1 253.9 mm to (-177.5, 121.9)
- moved J3 54.1 mm to (57.4, 108.4), turned to -90 degrees
- moved JP1 40.6 mm to (108.2, 132.7), turned to 0 degrees
- moved J7 35.3 mm to (85.8, 154.0), turned to 90 degrees
- moved C12 33.2 mm to (104.3, 111.7), turned to 90 degrees
- moved R20 30.7 mm to (104.3, 108.2), turned to 90 degrees
- moved R15 22.2 mm to (83.5, 121.3)
- moved R2 22.2 mm to (86.9, 133.2), turned to -90 degrees
- moved R3 22.2 mm to (81.2, 133.2), turned to -90 degrees
- moved R4 22.2 mm to (75.6, 133.2), turned to -90 degrees
- moved R5 22.2 mm to (70.0, 133.2), turned to -90 degrees
- moved R6 22.2 mm to (64.4, 133.2), turned to -90 degrees
- moved R10 21.2 mm to (101.0, 109.5)
- moved C10 20.5 mm to (76.0, 135.8), turned to 0 degrees
- moved R9 20.2 mm to (100.7, 111.7)
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- renumbered D2 to D1, D1 to D2, D20 to D3, D5 to D4, D4 to D6, D3 to D7, J10 to J1, J3 to J2, J4 to J3, J12 to J5, J9 to J6, J1 to J8, R7 to R1, R12 to R10, R9 to R11, R10 to R15, R14 to R16, R13 to R17, R15 to R18, R16 to R19, R1 to R2, R2 to R3, R3 to R4, R4 to R5, R5 to R6, R6 to R7, R11 to R9
Connections:
- C10 pad 1: +5V -> +3V3
- C11 pad 1: +5V -> Net-(C11-Pad1)
- C12 pad 1: +5V -> NRST
- C6 pad 1: Net-(C6-Pad1) -> /Buck Converter/VIN_12v
- C7 pad 1: Net-(C7-Pad1) -> +5V
- C8 pad 1: Net-(C7-Pad1) -> +3V3
- C9 pad 1: Net-(C7-Pad1) -> +3V3
- D2 pad 1: Net-(D1-Pad1) -> Net-(D2-Pad1)
- D4 pad 1: Net-(D1-Pad1) -> Net-(D2-Pad1)
- F1 pad 1: Net-(D1-Pad1) -> Net-(D2-Pad1)
- F1 pad 2: Net-(C6-Pad1) -> /Buck Converter/VIN_12v
- J1 pad 1: Net-(D1-Pad1) -> Net-(D2-Pad1)
- J1 pad 2: Net-(J10-Pad2) -> Net-(J1-Pad2)
- J4 pad 2: +5V -> GND
- J7 pad 1: VIN -> +3V3
- J7 pad 2: GND -> SWIM
- J7 pad 3: unconnected-(J7-Pad3) -> GND
- JP1 pad 1: Net-(JP1-Pad1) -> Net-(J1-Pad2)
- JP1 pad 2: +5V -> Net-(D2-Pad1)
- R1 pad 1: Net-(J10-Pad2) -> Net-(J1-Pad2)
- R11 pad 1: VIN_SENSE -> GND
- R11 pad 2: GND -> VIN_SENSE
- R20 pad 1: Net-(C6-Pad1) -> NRST
- R20 pad 2: Net-(R20-Pad2) -> +3V3
- R21 pad 1: Net-(R20-Pad2) -> /Buck Converter/VIN_12v
- R21 pad 2: GND -> Net-(R21-Pad2)
- R8 pad 1: Net-(D1-Pad1) -> VIN
- U6 pad 1: RESET -> GND
- U6 pad 2: VIN_SENSE -> +3V3
- U6 pad 3: UPS_SENSE -> +5V
- U7 pad 1: POW_ENABLE -> unconnected-(U7-Pad1)
- U7 pad 10: GND -> unconnected-(U7-Pad10)
- U7 pad 11: RS232_RXD -> I2C_SDA
- U7 pad 12: RS232_TXD -> I2C_SCL
- U7 pad 13: unconnected-(U9-Pad13) -> POW_ENABLE
- U7 pad 14: unconnected-(U9-Pad14) -> VOUT_SENSE
- U7 pad 15: VIN_SENSE -> Power_Button
- U7 pad 16: UPS_SENSE -> Spare_Button
- U7 pad 17: unconnected-(U9-Pad17) -> DEBUG_LED
- U7 pad 19: Power_Button -> UPS_SENSE
- U7 pad 2: unconnected-(U9-Pad2) -> RS232_TXD
- U7 pad 20: Spare_Button -> VIN_SENSE
- U7 pad 3: I2C_SDA -> RS232_RXD
- U7 pad 4: I2C_SCL -> NRST
- U7 pad 7: unconnected-(U9-Pad7) -> GND
- U7 pad 8: +5V -> Net-(C11-Pad1)
- U7 pad 9: Net-(TP1-Pad1) -> +3V3
Routing:
- net +5V: track 105.9 -> 0.00 mm, vias 5 -> 0
- net VIN: track 76.8 -> 0.00 mm
- net I2C_SDA: track 76.7 -> 0.00 mm, vias 2 -> 0
- net Net-(C1-Pad1): track 68.6 -> 0.00 mm, vias 1 -> 0
- net I2C_SCL: track 64.9 -> 0.00 mm, vias 2 -> 0
- net Power_Button: track 52.9 -> 0.00 mm, vias 4 -> 0
- net POW_OUT: track 52.2 -> 0.00 mm, vias 1 -> 0
- net Spare_Button: track 48.2 -> 0.00 mm, vias 3 -> 0
- net Net-(C1-Pad2): track 45.3 -> 0.00 mm
- net Net-(J10-Pad2): track 45.2 -> 0.00 mm
- net RS232_TXD: track 43.3 -> 0.00 mm, vias 1 -> 0
- net POW_ENABLE: track 41.2 -> 0.00 mm, vias 2 -> 0
- net VIN_SENSE: track 40.2 -> 0.00 mm, vias 1 -> 0
- net RS232_RXD: track 38.8 -> 0.00 mm, vias 1 -> 0
- net +3V3: track 38.5 -> 0.00 mm
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Other:
- board text removed: "POW EN"
