File: hw/v0p9p5/ras_pi_supercap_ups.kicad_pcb (KiCad board)
At the start: 2 copper layers, 65 x 56 mm, 83 parts, among them J1 Conn_01x03, J2 Conn_01x05, J3 Conn_01x03, J4 Force Power On, J5 171826-4, J6 LEDs and Buttons, J7 STLinkV2 Connector, J8 Raspberry_Pi_2_3, J9 Test Points, Q1 IRF5305, SW1 Reset, U1 KA431SMFTF, U2 KA431SMFTF, U3 KA431SMFTF, U4 KA431SMFTF, U5 KA431SMFTF, U6 AMS1117-3.3, U7 STM8S003F3P, U8 TPS54331DR

Commit message: Updates - candidate board layout
Parts:
- removed C6: 10u 25V X7R, Capacitor_SMD:C_0805_2012Metric
- added D9: Green, LED_SMD:LED_0805_2012Metric, F.Cu at (74.5, 131.7)
- added J10: Barrel_Jack, Connector_BarrelJack:BarrelJack_Wuerth_6941xx301002, F.Cu at (104.8, 112.4)
- added R27: 1k, Resistor_SMD:R_0805_2012Metric, F.Cu at (78.0, 131.7)
- J9: footprint Connector_PinHeader_1.00mm:PinHeader_1x03_P1.00mm_Vertical -> Connector_PinHeader_2.54mm:PinHeader_1x03_P2.54mm_Vertical
- JP1: moved to B.Cu
- moved R1 255.1 mm to (76.2, 148.3)
- moved SW1 55.1 mm to (62.7, 134.3), turned to 90 degrees
- moved R20 50.0 mm to (60.0, 131.4)
- moved C12 49.9 mm to (60.0, 134.8), turned to -90 degrees
- moved J9 30.8 mm to (101.3, 111.9)
- moved U5 29.1 mm to (90.6, 134.7)
- moved U4 27.0 mm to (94.1, 134.7)
- moved R6 26.9 mm to (91.2, 130.4), turned to 90 degrees
- moved U3 24.8 mm to (97.6, 134.7)
- moved R5 24.5 mm to (94.4, 130.4), turned to 90 degrees
- moved U2 22.7 mm to (101.1, 134.7)
- moved R4 22.1 mm to (97.6, 130.4), turned to 90 degrees
- moved R18 21.7 mm to (83.3, 135.5), turned to 180 degrees
- moved U1 20.6 mm to (104.6, 134.7)
- moved J7 20.4 mm to (78.3, 135.1), turned to -90 degrees
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Connections:
- C15 pad 1: /Buck Converter/VIN_12v -> +12V
- C16 pad 1: /Buck Converter/VIN_12v -> +12V
- C17 pad 1: /Buck Converter/VIN_12v -> +12V
- F1 pad 2: /Buck Converter/VIN_12v -> +12V
- J2 pad 3: unconnected-(J2-Pad3) -> PI_3v3
- J8 pad 1: +3V3 -> PI_3v3
- J8 pad 10: GPIO15 -> unconnected-(J8-Pad10)
- J8 pad 11: GPIO17 -> unconnected-(J8-Pad11)
- J8 pad 12: GPIO18 -> unconnected-(J8-Pad12)
- J8 pad 13: GPIO27 -> unconnected-(J8-Pad13)
- J8 pad 15: GPIO22 -> unconnected-(J8-Pad15)
- J8 pad 16: GPIO23 -> unconnected-(J8-Pad16)
- J8 pad 17: +3V3 -> PI_3v3
- J8 pad 18: GPIO24 -> unconnected-(J8-Pad18)
- J8 pad 19: GPIO10 -> unconnected-(J8-Pad19)
- J8 pad 21: GPIO9 -> unconnected-(J8-Pad21)
- J8 pad 22: GPIO25 -> unconnected-(J8-Pad22)
- J8 pad 23: GPIO11 -> unconnected-(J8-Pad23)
- J8 pad 24: GPIO8 -> unconnected-(J8-Pad24)
- J8 pad 26: GPIO7 -> unconnected-(J8-Pad26)
- J8 pad 27: GPIO0 -> unconnected-(J8-Pad27)
- J8 pad 28: GPIO1 -> unconnected-(J8-Pad28)
- J8 pad 29: GPIO5 -> unconnected-(J8-Pad29)
- J8 pad 31: GPIO6 -> unconnected-(J8-Pad31)
- J8 pad 32: GPIO12 -> unconnected-(J8-Pad32)
- J8 pad 33: GPIO13 -> unconnected-(J8-Pad33)
- J8 pad 35: GPIO19 -> unconnected-(J8-Pad35)
- J8 pad 36: GPIO16 -> unconnected-(J8-Pad36)
- J8 pad 37: GPIO26 -> unconnected-(J8-Pad37)
- J8 pad 38: GPIO20 -> unconnected-(J8-Pad38)
- J8 pad 40: GPIO21 -> unconnected-(J8-Pad40)
- J8 pad 7: GPIO4 -> unconnected-(J8-Pad7)
- J8 pad 8: GPIO14 -> unconnected-(J8-Pad8)
- R18 pad 1: +5V -> +3V3
- R19 pad 1: +5V -> +3V3
- R21 pad 1: /Buck Converter/VIN_12v -> +12V
- U7 pad 18: unconnected-(U7-Pad18) -> SWIM
- U8 pad 2: /Buck Converter/VIN_12v -> +12V
Routing:
- net GND: track 0.00 -> 102.9 mm, vias 0 -> 14
- net +5V: track 0.00 -> 93.6 mm, vias 0 -> 4
- net Power_Button: track 0.00 -> 71.2 mm, vias 0 -> 3
- net Net-(D6-Pad2): track 0.00 -> 69.4 mm, vias 0 -> 2
- net Spare_Button: track 0.00 -> 62.3 mm, vias 0 -> 3
- net Net-(J1-Pad2): track 0.00 -> 61.7 mm, vias 0 -> 1
- net +3V3: track 0.00 -> 61.0 mm, vias 0 -> 5
- net Net-(C1-Pad1): track 0.00 -> 56.1 mm, vias 0 -> 2
- net Net-(C4-Pad2): track 0.00 -> 45.3 mm
- net I2C_SCL: track 0.00 -> 42.3 mm, vias 0 -> 1
- net Net-(D5-Pad2): track 0.00 -> 41.2 mm, vias 0 -> 2
- net PI_3v3: track 0.00 -> 40.6 mm
- net VIN_SENSE: track 0.00 -> 40.0 mm, vias 0 -> 2
- net Net-(D2-Pad1): track 0.00 -> 39.3 mm, vias 0 -> 2
- net I2C_SDA: track 0.00 -> 39.2 mm, vias 0 -> 1
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Other:
- board text added: "12v"
- board text added: "3.3v"
- board text added: "3v3"
- board text added: "Barrel Jack"
- board text added: "Based upon: - 12v SuperCapacitor UPS - Scott Baker - http://www.smbaker.com - MFM Emulator - David Gesswein - https://www.pdp8online.com/mfm/"
- board text added: "Berg Connector"
- board text added: "Cut to enable discharge circuit"
- board text added: "HOT!"
- board text added: "NC"
- board text added: "NRST"
- board text added: "POW ENB Override"
- board text added: "PWR Button"
- board text added: "RESET"
- board text added: "STLinkV2"
- board text added: "SUPER UPS"
- board text added: "SWIM"
- board text added: "SuperUPS for Raspberry Pi v0.9.5"
- board text added: "UART1"
- board text added: "[Optional]"
- board text added: "for Raspberry Pi v0.9.5"
- board text added: "https://github.com/akuker/SuperUPS"
- board text removed: "RST"
- board text removed: "Raspberry Pi 12v UPS v0.9"
- board text removed: "https://github.com/akuker/hw_projects"
- board text removed: "https://github.com/akuker/hw_projects Based upon designs: Scott Baker - 12v SuperCapacitor UPS - http://www.smbaker.com David Gesswein - MFM Emulator - https://www.pdp8online.com/mfm/"

Commit message: updates
Parts:
- turned D1 to 90 degrees
- turned D7 to 180 degrees
Connections:
- D1 pad 1: GND -> VIN
- D1 pad 2: VIN -> GND
- D7 pad 1: GND -> POW_OUT
- D7 pad 2: POW_OUT -> GND
Other:
- board text added: "Aux Button"
Changed lines of the file:
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@@
   )
   (footprint "Diode_SMD:D_SOD-323" (layer "F.Cu")
-    (at 101.9 120.6 -90)
+    (at 101.9 120.6 90)
     (descr "SOD-323")
     (tags "SOD-323")
@@
     (fp_line (start -0.9 0.7) (end -0.9 -0.7) (layer "F.Fab") (width 0.1))
     (fp_line (start -0.9 -0.7) (end 0.9 -0.7) (layer "F.Fab") (width 0.1))
-    (pad "1" smd rect (at -1.05 0 270) (size 0.6 0.45) (layers "F.Cu" "F.Paste" "F.Mask")
-      (net 2 "GND") (pinfunction "A1") (pintype "passive"))
-    (pad "2" smd rect (at 1.05 0 270) (size 0.6 0.45) (layers "F.Cu" "F.Paste" "F.Mask")
-      (net 1 "VIN") (pinfunction "A2") (pintype "passive"))
+    (pad "1" smd rect (at -1.05 0 90) (size 0.6 0.45) (layers "F.Cu" "F.Paste" "F.Mask")
+      (net 1 "VIN") (pinfunction "A1") (pintype "passive"))
+    (pad "2" smd rect (at 1.05 0 90) (size 0.6 0.45) (layers "F.Cu" "F.Paste" "F.Mask")
+      (net 2 "GND") (pinfunction "A2") (pintype "passive"))
     (model "${KICAD6_3DMODEL_DIR}/Diode_SMD.3dshapes/D_SOD-323.wrl"
       (offset (xyz 0 0 0))
@@
   )
   (footprint "Diode_SMD:D_SOD-323" (layer "F.Cu")
-    (at 64.8 108.41)
+    (at 64.8 108.41 180)
     (descr "SOD-323")
     (tags "SOD-323")
@@
     (property "Sheetname" "")
     (attr smd)
-    (fp_text reference "D7" (at -0.1 -1.51 180) (layer "F.SilkS")
+    (fp_text reference "D7" (at -0.1 -1.51) (layer "F.SilkS")
       (effects (font (size 0.7 0.7) (thickness 0.1)))
     )
@@
     (fp_line (start -0.9 0.7) (end -0.9 -0.7) (layer "F.Fab") (width 0.1))
     (fp_line (start -0.3 0) (end -0.5 0) (layer "F.Fab") (width 0.1))
-    (pad "1" smd rect (at -1.05 0) (size 0.6 0.45) (layers "F.Cu" "F.Paste" "F.Mask")
-      (net 2 "GND") (pinfunction "A1") (pintype "passive"))
-    (pad "2" smd rect (at 1.05 0) (size 0.6 0.45) (layers "F.Cu" "F.Paste" "F.Mask")
-      (net 3 "POW_OUT") (pinfunction "A2") (pintype "passive"))
+    (pad "1" smd rect (at -1.05 0 180) (size 0.6 0.45) (layers "F.Cu" "F.Paste" "F.Mask")
+      (net 3 "POW_OUT") (pinfunction "A1") (pintype "passive"))
+    (pad "2" smd rect (at 1.05 0 180) (size 0.6 0.45) (layers "F.Cu" "F.Paste" "F.Mask")
+      (net 2 "GND") (pinfunction "A2") (pintype "passive"))
     (model "${KICAD6_3DMODEL_DIR}/Diode_SMD.3dshapes/D_SOD-323.wrl"
       (offset (xyz 0 0 0))
@@
       (effects (font (size 1.003283 1.003283) (thickness 0.15)))
     )
-    (fp_text user "+5" (at 3.7 -6 90 unlocked) (layer "F.SilkS")
+    (fp_text user "GND" (at 1.3 -6 90 unlocked) (layer "F.SilkS")
       (effects (font (size 0.7 0.7) (thickness 0.1)))
     )
@@
       (effects (font (size 0.7 0.7) (thickness 0.1)))
     )
-    (fp_text user "GND" (at 1.3 -6 90 unlocked) (layer "F.SilkS")
+    (fp_text user "+5" (at 3.7 -6 90 unlocked) (layer "F.SilkS")
       (effects (font (size 0.7 0.7) (thickness 0.1)))
     )
@@
       (effects (font (size 0.7 0.7) (thickness 0.1)))
     )
-    (fp_line (start -5 -6.75) (end 5 -6.75) (layer "F.SilkS") (width 0.127))
     (fp_line (start 5 -6.75) (end 5 -2.15) (layer "F.SilkS") (width 0.127))
-    (fp_line (start 5 -0.75) (end 5 6.75) (layer "F.SilkS") (width 0.127))
     (fp_line (start -5 -0.75) (end -5 -2.15) (layer "F.SilkS") (width 0.127))
     (fp_line (start -5 -2.15) (end 5 -2.15) (layer "F.SilkS") (width 0.127))
-    (fp_line (start 5 6.75) (end -5 6.75) (layer "F.SilkS") (width 0.127))
+    (fp_line (start -5 6.75) (end -5 -0.75) (layer "F.SilkS") (width 0.127))
+    (fp_line (start 5 -2.15) (end 5 -0.75) (layer "F.SilkS") (width 0.127))
     (fp_line (start -5 -2.15) (end -5 -6.75) (layer "F.SilkS") (width 0.127))
+    (fp_line (start 5 -0.75) (end 5 6.75) (layer "F.SilkS") (width 0.127))
     (fp_line (start -5 -0.75) (end 5 -0.75) (layer "F.SilkS") (width 0.127))
-    (fp_line (start 5 -2.15) (end 5 -0.75) (layer "F.SilkS") (width 0.127))
-    (fp_line (start -5 6.75) (end -5 -0.75) (layer "F.SilkS") (width 0.127))
+    (fp_line (start -5 -6.75) (end 5 -6.75) (layer "F.SilkS") (width 0.127))
+    (fp_line (start 5 6.75) (end -5 6.75) (layer "F.SilkS") (width 0.127))
     (fp_circle (center -5.8 -5) (end -5.7 -5) (layer "F.SilkS") (width 0.2) (fill none))
-    (fp_line (start -5.25 -7) (end 5.25 -7) (layer "F.CrtYd") (width 0.05))
-    (fp_line (start 5.25 -7) (end 5.25 7) (layer "F.CrtYd") (width 0.05))
     (fp_line (start 5.25 7) (end -5.25 7) (layer "F.CrtYd") (width 0.05))
     (fp_line (start -5.25 7) (end -5.25 -7) (layer "F.CrtYd") (width 0.05))
+    (fp_line (start -5.25 -7) (end 5.25 -7) (layer "F.CrtYd") (width 0.05))
+    (fp_line (start 5.25 -7) (end 5.25 7) (layer "F.CrtYd") (width 0.05))
+    (fp_line (start 5 6.75) (end -5 6.75) (layer "F.Fab") (width 0.127))
     (fp_line (start -5 6.75) (end -5 -6.75) (layer "F.Fab") (width 0.127))
     (fp_line (start 5 6.75) (end 5 -6.75) (layer "F.Fab") (width 0.127))
     (fp_line (start -5 -6.75) (end 5 -6.75) (layer "F.Fab") (width 0.127))
-    (fp_line (start 5 6.75) (end -5 6.75) (layer "F.Fab") (width 0.127))
     (pad "1" thru_hole rect (at -3.75 -4.55 90) (size 1.408 1.408) (drill 0.9) (layers *.Cu *.Mask)
       (net 1 "VIN") (pinfunction "Pin_1") (pintype "passive"))
@@
     (property "Sheetname" "")
     (attr through_hole)
-    (fp_text reference "J6" (at 0.76 9.605 -90) (layer "F.SilkS")
+    (fp_text reference "J6" (at 1.06 -3.195 -90) (layer "F.SilkS")
       (effects (font (size 0.7 0.7) (thickness 0.1)))
     )
@@
     (pad "8" smd roundrect locked (at 2.47 -1.905 180) (size 1.97 0.6) (layers "F.Cu" "F.Paste" "F.Mask") (roundrect_rratio 0.07)
       (net 27 "Net-(C18-Pad1)") (pinfunction "PH") (pintype "input"))
+    (model "${KICAD6_3DMODEL_DIR}/Package_SO.3dshapes/SOIC-8_3.9x4.9mm_P1.27mm.wrl"
+      (offset (xyz 0 0 0))
+      (scale (xyz 1 1 1))
+      (rotate (xyz 0 0 0))
+    )
   )
   (footprint "Package_TO_SOT_SMD:SOT-23" (layer "F.Cu")
@@
   (gr_line (start 111.1 131.033) (end 111.1 136.367) (layer "B.SilkS") (width 0.15))
   (gr_rect (start 60.706 123.434) (end 55.86 110.434) (layer "B.SilkS") (width 0.15) (fill none))
-  (gr_rect (start 80.8 145.5) (end 97.1 153.6) (layer "B.SilkS") (width 0.2) (fill none))
+  (gr_rect (start 84.2 151.2) (end 92.8 153.6) (layer "B.SilkS") (width 0.2) (fill none))
   (gr_rect (start 97.6 110.6) (end 102.5 118.6) (layer "B.SilkS") (width 0.15) (fill none))
   (gr_rect (start 54.864 123.556) (end 50.8 134.112) (layer "B.SilkS") (width 0.15) (fill none))
@@
   (gr_rect (start 50.8 110.49) (end 54.864 123.556) (layer "B.SilkS") (width 0.15) (fill none))
   (gr_rect (start 102.1 151.2) (end 108.4 155.4) (layer "B.SilkS") (width 0.15) (fill none))
+  (gr_rect (start 95.65 151.2) (end 101.95 155.4) (layer "B.SilkS") (width 0.15) (fill none))
   (gr_line (start 55.77 134.3) (end 50.8 134.3) (layer "F.SilkS") (width 0.15))
   (gr_rect (start 69.1 132.7) (end 79.879937 137.607) (layer "F.SilkS") (width 0.15) (fill none))
@@
   (gr_line (start 55.77 130.195) (end 55.77 134.3) (layer "F.SilkS") (width 0.15))
   (gr_rect (start 102.1 155.4) (end 108.4 151.2) (layer "F.SilkS") (width 0.15) (fill none))
+  (gr_rect (start 95.65 155.4) (end 101.95 151.2) (layer "F.SilkS") (width 0.15) (fill none))
   (gr_line (start 58.5 136.7) (end 58.5 130.2) (layer "F.SilkS") (width 0.15))
   (gr_line locked (start 115 103.5) (end 115 152.5) (layer "Edge.Cuts") (width 0.1))
@@
     (effects (font (size 0.7 0.7) (thickness 0.1) italic) (justify mirror))
   )
+  (gr_text "Aux Button" (at 101.7 152.2) (layer "B.SilkS")
+    (effects (font (size 0.7 0.7) (thickness 0.1)) (justify left mirror))
+  )
   (gr_text "RXD" (at 51.5 127.2 270) (layer "B.SilkS")
     (effects (font (size 0.7 0.7) (thickness 0.1)) (justify mirror))
@@
     (effects (font (size 3 3) (thickness 0.5) italic))
   )
+  (gr_text "Aux Button" (at 95.9 152.2) (layer "F.SilkS")
+    (effects (font (size 0.7 0.7) (thickness 0.1)) (justify left))
+  )
   (gr_text "GND" (at 51.562 119.888 270) (layer "F.SilkS")
