File: hw/v0p9p5/ras_pi_supercap_ups.kicad_sch (KiCad schematic)
At the start: 63 parts, among them J10 Conn_01x03, J12 171826-4, J3 Conn_01x05, J4 Conn_01x03, J6 Conn_01x04, J7 Conn_01x03, J8 Conn_02x03_Odd_Even, J9 LEDs and Buttons, Q1 IRF5305, U1 KA431SMFTF, U2 KA431SMFTF, U3 KA431SMFTF, U4 KA431SMFTF, U5 KA431SMFTF, U6 LM2596S-5, U7 L7805, U8 ATtiny85-20P, U9 STC8H1K08

Commit message: updates... pulled in buck conv
Parts:
- removed C10, C11, C7, C8, C9: 22u 10V X7R, Capacitor_SMD:C_0805_2012Metric, symbol Device:C_Polarized_Small_US
- removed C12: 0.1u, Capacitor_SMD:C_0805_2012Metric, symbol Device:C_Polarized_Small_US
- removed J6: Conn_01x04, Connector_PinHeader_2.54mm:PinHeader_1x04_P2.54mm_Vertical, symbol Connector_Generic:Conn_01x04
- removed J7: Conn_01x03, Connector_PinHeader_2.54mm:PinHeader_1x03_P2.54mm_Vertical, symbol Connector_Generic:Conn_01x03
- removed JP1, JP2, JP3: SolderJumper_2_Open, Jumper:SolderJumper-2_P1.3mm_Open_RoundedPad1.0x1.5mm, symbol Jumper:SolderJumper_2_Open
- removed R21: 47k, Resistor_SMD:R_0805_2012Metric, symbol Device:R_Small
- removed TP1: TestPoint_Small, TestPoint:TestPoint_THTPad_D1.0mm_Drill0.5mm, symbol Connector:TestPoint_Small
- removed U6: LM2596S-5, Package_TO_SOT_SMD:TO-263-5_TabPin3, symbol Regulator_Switching:LM2596S-5
- removed U7: L7805, Connector_PinSocket_2.54mm:PinSocket_1x03_P2.54mm_Vertical, symbol Regulator_Linear:L7805
- removed U8: ATtiny85-20P, Package_DIP:DIP-8_W7.62mm, symbol MCU_Microchip_ATtiny:ATtiny85-20P
- removed U9: STC8H1K08, Package_SO:TSSOP-20_4.4x6.5mm_P0.65mm, symbol supercap_library:STC8H1K08
- added C10, C11, C12, C7, C8, C9: (no value), symbol Device:C_Small
- added D5: (no value), symbol Device:LED_Small
- added J7: (no value), symbol Connector_Generic:Conn_01x04
- added JP1: (no value), symbol Jumper:SolderJumper_2_Bridged
- added R12, R13, R14: (no value), symbol Device:R_Small
- added SW1: (no value), symbol Switch:SW_Push
- added U6: (no value), symbol Regulator_Linear:AMS1117-3.3
- added U7: (no value), symbol MCU_ST_STM8:STM8S003F3P
- C1, C2, C3, C4, C5: value 10F -> (none); footprint Capacitor_THT:CP_Radial_D12.5mm_P5.00mm -> (none)
- C6: value 10u 25V X7R -> (none); footprint Capacitor_SMD:C_0805_2012Metric -> (none); symbol Device:C_Polarized_Small_US -> Device:C_Small
- D1: renamed from D2; value PTVSHC3D15VUH -> (none); footprint Diode_SMD:D_SOD-323 -> (none)
- D2: renamed from D1; value B340LA-13-F -> (none); footprint Diode_SMD:D_SMA -> (none)
- D3: renamed from D20; value Green -> (none); footprint LED_SMD:LED_0805_2012Metric -> (none)
- D4: renamed from D5; value B340LA-13-F -> (none); footprint Diode_SMD:D_SMA -> (none)
- D6: renamed from D4; value Green -> (none); footprint LED_SMD:LED_0805_2012Metric -> (none)
- D7: renamed from D3; value PTVSHC3D15VUH -> (none); footprint Diode_SMD:D_SOD-323 -> (none)
- F1: value Fuse_Small -> (none); footprint Fuse:Fuse_1206_3216Metric -> (none)
- H1, H2, H3, H4: value MountingHole -> (none); footprint MountingHole:MountingHole_2.7mm_M2.5 -> (none)
- J1: renamed from J10; value Conn_01x03 -> (none); footprint Connector_PinHeader_2.54mm:PinHeader_1x03_P2.54mm_Vertical -> (none)
- J2: renamed from J3; value Conn_01x05 -> (none); footprint Connector_PinHeader_2.54mm:PinHeader_1x05_P2.54mm_Vertical -> (none)
- J3: renamed from J4; value Conn_01x03 -> (none); footprint Connector_PinHeader_2.54mm:PinHeader_1x03_P2.54mm_Vertical -> (none)
- J4: renamed from J8; value Conn_02x03_Odd_Even -> (none); footprint Connector_PinHeader_2.54mm:PinHeader_2x03_P2.54mm_Vertical -> (none); symbol Connector_Generic:Conn_02x03_Odd_Even -> Connector_Generic:Conn_01x02
- J5: renamed from J12; value 171826-4 -> (none); footprint TE_171826-4 -> (none)
- J6: renamed from J9; value LEDs and Buttons -> (none); footprint Connector_PinHeader_2.54mm:PinHeader_1x04_P2.54mm_Vertical -> (none)
- Q1: value IRF5305 -> (none); footprint Package_TO_SOT_SMD:TO-263-2 -> (none)
- R1: renamed from R7; value 10 3W -> (none); footprint Resistor_THT:R_Axial_DIN0516_L15.5mm_D5.0mm_P25.40mm_Horizontal -> (none)
- R10: renamed from R12; value 2.2k -> (none); footprint Resistor_SMD:R_0805_2012Metric -> (none)
- R11: renamed from R9; value 2.2k -> (none); footprint Resistor_SMD:R_0805_2012Metric -> (none)
- R15: renamed from R10; value 1k -> (none); footprint Resistor_SMD:R_0805_2012Metric -> (none)
- R16: renamed from R14; value 10k -> (none); footprint Resistor_SMD:R_0805_2012Metric -> (none)
- R17: renamed from R13; value 1k -> (none); footprint Resistor_SMD:R_0805_2012Metric -> (none)
- R18: renamed from R15; value 1k -> (none); footprint Resistor_SMD:R_0805_2012Metric -> (none)
- R19: renamed from R16; value 1k -> (none); footprint Resistor_SMD:R_0805_2012Metric -> (none)
- R2: renamed from R1; value 1k -> (none); footprint Resistor_SMD:R_1206_3216Metric -> (none)
- R20: value 47k -> (none); footprint Resistor_SMD:R_0805_2012Metric -> (none); DigikeyPN CF14JT47K0TR-ND -> CF14JT10K0CT-ND; LCSC C17713 -> C17414
- R3: renamed from R2; value 1k -> (none); footprint Resistor_SMD:R_1206_3216Metric -> (none)
- R4: renamed from R3; value 1k -> (none); footprint Resistor_SMD:R_1206_3216Metric -> (none)
- R5: renamed from R4; value 1k -> (none); footprint Resistor_SMD:R_1206_3216Metric -> (none)
- R6: renamed from R5; value 1k -> (none); footprint Resistor_SMD:R_1206_3216Metric -> (none)
- R7: renamed from R6; value 1k -> (none); footprint Resistor_SMD:R_0805_2012Metric -> (none)
- R8: value 10k -> (none); footprint Resistor_SMD:R_0805_2012Metric -> (none)
- R9: renamed from R11; value 10k -> (none); footprint Resistor_SMD:R_0805_2012Metric -> (none)
- U1, U2, U3, U4, U5: value KA431SMFTF -> (none); footprint Package_TO_SOT_SMD:SOT-23 -> (none)
Connections:
- net +5V: now also C7.1, R12.1, U6.3 (VI); no longer J4.2 (Pin_2)
- net GND: now also J4.2 (Pin_2), R11.1, C10.2, C11.2, C12.2, C7.2, C8.2, C9.2, D5.1 (K), J7.3 (Pin_3), R13.2, SW1.1, U6.1 (GND), U7.7 (VSS); no longer J4.6 (Pin_6), R11.2
- net I2C_SCL: now also U7.12 (PB4); no longer J4.3 (Pin_3)
- net I2C_SDA: now also U7.11 (PB5); no longer J4.4 (Pin_4)
- net POW_ENABLE: now also U7.13 (PC3)
- net Power_Button: now also U7.15 (PC5)
- net RS232_RXD: now also U7.3 (PD6)
- net RS232_TXD: now also U7.2 (PD5)
- net Spare_Button: now also U7.16 (PC6)
- net UPS_SENSE: now also U7.19 (PD2)
- net VIN: now also R8.1
- net VIN_SENSE: now also R11.2, U7.20 (PD3); no longer R11.1
- net at D2.1 (K), D4.1 (K), F1.1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: now also JP1.2 (B); no longer R8.1
- net at J1.2 (Pin_2), R1.1: now also JP1.1 (A)
- net Buck Converter/VIN_12v: now reaches C6.1, F1.2
- net Buck Converter/VIN_12v: no longer R20.1
- net +3V3: now reaches R20.2
- net +3V3: now also C10.1, C8.1, C9.1, J7.1 (Pin_1), R14.1, U6.2 (VO), U7.9 (VDD)
- removed net RESET: J4.5 (Pin_5)
- new net: C11.1, U7.8 (VCAP)
- new net: D5.2 (A), R14.2
- new net DEBUG_LED: U7.17 (PC7)
- new net NRST: C12.1, J7.4 (Pin_4), R20.1, SW1.2, U7.4 (NRST)
- new net SWIM: J7.2 (Pin_2)
- new net VOUT_SENSE: R12.2, R13.1, U7.14 (PC4)
- no-connect marks 11 -> 2
Other:
- added sheet Buck Converter (12v_buck_converter.kicad_sch)
- note removed: "Option 1 - LM2596S"
- note removed: "Option 2 - L7805"
- moved on the sheet: D6, D7, J2, J5, J6, R11, R15, R18, R19, R8
