File: hw/v0p9p5/ras_pi_supercap_ups.kicad_sch (KiCad schematic)
At the start: 61 parts

Commit message: Updates - candidate board layout
Parts:
- removed C6: (no value), symbol Device:C_Small
- added D9: Green, LED_SMD:LED_0805_2012Metric, symbol Device:LED_Small
- added J10: Barrel_Jack, Connector_BarrelJack:BarrelJack_Wuerth_6941xx301002, symbol Connector:Barrel_Jack_Switch
- added R27: 1k, Resistor_SMD:R_0805_2012Metric, symbol Device:R_Small
- C1, C2, C3, C4, C5: value (none) -> 10F; footprint (none) -> Capacitor_THT:CP_Radial_D12.5mm_P5.00mm
- C10, C7, C8: value (none) -> 10u; footprint (none) -> Capacitor_SMD:C_0805_2012Metric
- C11, C12: value (none) -> 1u; footprint (none) -> Capacitor_SMD:C_0805_2012Metric
- C9: value (none) -> 100n; footprint (none) -> Capacitor_SMD:C_0805_2012Metric
- D1, D7: value (none) -> PTVSHC3D15VUH; footprint (none) -> Diode_SMD:D_SOD-323
- D2, D4: value (none) -> B340LA-13-F; footprint (none) -> Diode_SMD:D_SMA
- D3, D5, D6: value (none) -> Green; footprint (none) -> LED_SMD:LED_0805_2012Metric
- F1: value (none) -> Fuse_Small; footprint (none) -> Fuse:Fuse_1206_3216Metric
- H1, H2, H3, H4: value (none) -> MountingHole; footprint (none) -> MountingHole:MountingHole_2.7mm_M2.5
- J1, J3: value (none) -> Conn_01x03; footprint (none) -> Connector_PinHeader_2.54mm:PinHeader_1x03_P2.54mm_Vertical
- J2: value (none) -> Conn_01x05; footprint (none) -> Connector_PinHeader_2.54mm:PinHeader_1x05_P2.54mm_Vertical
- J4: value (none) -> Force Power On; footprint (none) -> Connector_PinHeader_2.54mm:PinHeader_1x02_P2.54mm_Vertical
- J5: value (none) -> 171826-4; footprint (none) -> TE_171826-4; symbol 171826-4:171826-4 -> Connector_Generic:Conn_01x04
- J6: value (none) -> LEDs and Buttons; footprint (none) -> Connector_PinHeader_2.54mm:PinHeader_1x04_P2.54mm_Vertical
- J7: value (none) -> STLinkV2 Connector; footprint (none) -> Connector_PinHeader_2.54mm:PinHeader_1x04_P2.54mm_Vertical
- JP1: value (none) -> Charge Enb; footprint (none) -> Jumper:SolderJumper-2_P1.3mm_Bridged_RoundedPad1.0x1.5mm
- Q1: value (none) -> IRF5305; footprint (none) -> Package_TO_SOT_SMD:TO-263-2
- R1: value (none) -> 10 3W; footprint (none) -> Resistor_THT:R_Axial_DIN0516_L15.5mm_D5.0mm_P25.40mm_Horizontal
- R10, R11, R13: value (none) -> 2.2k; footprint (none) -> Resistor_SMD:R_0805_2012Metric
- R12, R16, R20, R8, R9: value (none) -> 10k; footprint (none) -> Resistor_SMD:R_0805_2012Metric
- R14, R15, R17, R18, R19, R7: value (none) -> 1k; footprint (none) -> Resistor_SMD:R_0805_2012Metric
- R2, R3, R4, R5, R6: value (none) -> 1k; footprint (none) -> Resistor_SMD:R_1206_3216Metric
- SW1: value (none) -> Reset; footprint (none) -> Button_Switch_THT:SW_PUSH_6mm_H4.3mm
- U1, U2, U3, U4, U5: value (none) -> KA431SMFTF; footprint (none) -> Package_TO_SOT_SMD:SOT-23
- U6: value (none) -> AMS1117-3.3; footprint (none) -> Package_TO_SOT_SMD:SOT-223-3_TabPin2
- U7: value (none) -> STM8S003F3P; footprint (none) -> Package_SO:TSSOP-20_4.4x6.5mm_P0.65mm
Connections:
- net +3V3: now also R18.1, R19.1, R27.1
- net +5V: no longer R18.1, R19.1
- net DEBUG_LED: now also D9.1 (K)
- net GND: now also J10.2, J10.3
- net SWIM: now also U7.18 (PD1)
- net VIN: now also J10.1
- net PI_3v3: now reaches J2.3 (Pin_3)
- net Buck Converter/VIN_12v renamed +12V
- new net: D9.2 (A), R27.2
- no-connect marks 2 -> 5
Other:
- moved on the sheet: J5

Commit message: updates
Connections:
- net GND: now also D1.2 (A2), D7.2 (A2); no longer D1.1 (A1), D7.1 (A1)
- net POW_OUT: now also D7.1 (A1); no longer D7.2 (A2)
- net VIN: now also D1.1 (A1); no longer D1.2 (A2)
Other:
- moved on the sheet: D1, D7
Changed lines of the file:
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@@
     (stroke (width 0) (type default) (color 0 0 0 0))
   )
-  (wire (pts (xy 321.31 88.9) (xy 321.31 91.44))
+  (wire (pts (xy 265.43 139.7) (xy 265.43 142.24))
     (stroke (width 0) (type default) (color 0 0 0 0))
   )
@@
     (stroke (width 0) (type default) (color 0 0 0 0))
   )
-  (wire (pts (xy 321.31 99.06) (xy 321.31 101.6))
+  (wire (pts (xy 265.43 149.86) (xy 265.43 152.4))
     (stroke (width 0) (type default) (color 0 0 0 0))
   )
@@
     (effects (font (size 1.27 1.27)) (justify left bottom))
   )
-  (global_label "POW_OUT" (shape input) (at 321.31 88.9 90) (fields_autoplaced)
-    (effects (font (size 1.27 1.27)) (justify left))
-    (property "Intersheet References" "${INTERSHEET_REFS}" (id 0) (at 321.2306 77.8388 90)
+  (global_label "POW_OUT" (shape input) (at 265.43 139.7 90) (fields_autoplaced)
+    (effects (font (size 1.27 1.27)) (justify left))
+    (property "Intersheet References" "${INTERSHEET_REFS}" (id 0) (at 265.3506 128.6388 90)
       (effects (font (size 1.27 1.27)) (justify left) hide)
     )
@@
     )
   )
-  (symbol (lib_id "power:GND") (at 321.31 101.6 0) (unit 1)
+  (symbol (lib_id "power:GND") (at 265.43 152.4 0) (unit 1)
     (in_bom yes) (on_board yes)
-    (property "Reference" "#PWR033" (id 0) (at 321.31 107.95 0)
-      (effects (font (size 1.27 1.27)) hide)
-    )
-    (property "Value" "GND" (id 1) (at 321.31 109.22 90)
-      (effects (font (size 1.27 1.27)) (justify left))
-    )
-    (property "Footprint" "" (id 2) (at 321.31 101.6 0)
-      (effects (font (size 1.27 1.27)) hide)
-    )
-    (property "Datasheet" "" (id 3) (at 321.31 101.6 0)
+    (property "Reference" "#PWR033" (id 0) (at 265.43 158.75 0)
+      (effects (font (size 1.27 1.27)) hide)
+    )
+    (property "Value" "GND" (id 1) (at 265.43 160.02 90)
+      (effects (font (size 1.27 1.27)) (justify left))
+    )
+    (property "Footprint" "" (id 2) (at 265.43 152.4 0)
+      (effects (font (size 1.27 1.27)) hide)
+    )
+    (property "Datasheet" "" (id 3) (at 265.43 152.4 0)
       (effects (font (size 1.27 1.27)) hide)
     )
@@
     (pin "1")
   )
-  (symbol (lib_id "Device:D_TVS") (at 41.91 43.18 90) (unit 1)
+  (symbol (lib_id "Device:D_TVS") (at 41.91 43.18 270) (unit 1)
     (in_bom yes) (on_board yes)
-    (property "Reference" "D1" (id 0) (at 44.45 41.9099 90)
+    (property "Reference" "D1" (id 0) (at 39.37 44.4501 90)
       (effects (font (size 1.27 1.27)) (justify right))
     )
-    (property "Value" "PTVSHC3D15VUH" (id 1) (at 24.13 43.18 90)
+    (property "Value" "PTVSHC3D15VUH" (id 1) (at 59.69 43.18 90)
       (effects (font (size 1.27 1.27)) (justify right) hide)
     )
@@
     (pin "2")
   )
-  (symbol (lib_id "Device:D_TVS") (at 321.31 95.25 90) (unit 1)
-    (in_bom yes) (on_board yes) (fields_autoplaced)
-    (property "Reference" "D7" (id 0) (at 323.85 93.9799 90)
-      (effects (font (size 1.27 1.27)) (justify right))
-    )
-    (property "Value" "PTVSHC3D15VUH" (id 1) (at 323.85 96.5199 90)
-      (effects (font (size 1.27 1.27)) (justify right))
-    )
-    (property "Footprint" "Diode_SMD:D_SOD-323" (id 2) (at 321.31 95.25 0)
-      (effects (font (size 1.27 1.27)) hide)
-    )
-    (property "Datasheet" "https://datasheet.lcsc.com/lcsc/1811091226_Shanghai-Prisemi-Elec-PTVSHC3D15VUH_C312234.pdf" (id 3) (at 321.31 95.25 0)
-      (effects (font (size 1.27 1.27)) hide)
-    )
-    (property "LCSC" "C312234" (id 4) (at 321.31 95.25 0)
-      (effects (font (size 1.27 1.27)) hide)
-    )
-    (property "DigikeyPN" "" (id 5) (at 321.31 95.25 0)
-      (effects (font (size 1.27 1.27)) hide)
-    )
+  (symbol (lib_id "Device:D_TVS") (at 265.43 146.05 270) (unit 1)
+    (in_bom yes) (on_board yes) (fields_autoplaced)
+    (property "Reference" "D7" (id 0) (at 267.97 144.7799 90)
+      (effects (font (size 1.27 1.27)) (justify left))
+    )
+    (property "Value" "PTVSHC3D15VUH" (id 1) (at 267.97 147.3199 90)
+      (effects (font (size 1.27 1.27)) (justify left))
+    )
+    (property "Footprint" "Diode_SMD:D_SOD-323" (id 2) (at 265.43 146.05 0)
+      (effects (font (size 1.27 1.27)) hide)
+    )
+    (property "Datasheet" "https://datasheet.lcsc.com/lcsc/1811091226_Shanghai-Prisemi-Elec-PTVSHC3D15VUH_C312234.pdf" (id 3) (at 265.43 146.05 0)
+      (effects (font (size 1.27 1.27)) hide)
+    )
+    (property "LCSC" "C312234" (id 4) (at 265.43 146.05 0)
+      (effects (font (size 1.27 1.27)) hide)
+    )
+    (property "DigikeyPN" "" (id 5) (at 265.43 146.05 0)
+      (effects (font (size 1.27 1.27)) hide)
+    )
