File: hw/v0p9p5/raspi_connectors.kicad_sch (KiCad schematic)
At the start: 2 parts, among them J1 Raspberry_Pi_2_3, J2 Raspberry_Pi_2_3

Commit message: updates... pulled in buck conv
Parts:
- removed J2: Raspberry_Pi_2_3, Connector_PinSocket_2.54mm:PinSocket_2x20_P2.54mm_Vertical, symbol Connector:Raspberry_Pi_2_3
- added C13: 10u, Capacitor_SMD:C_0805_2012Metric, symbol Device:C_Small
- added C14: 100n, Capacitor_SMD:C_0805_2012Metric, symbol Device:C_Small
- J8: renamed from J1; value Raspberry_Pi_2_3 -> (none); footprint Connector_PinSocket_2.54mm:PinSocket_2x20_P2.54mm_Vertical -> (none)
Connections:
- net GND: now also C13.2, C14.2
- net POW_OUT: now also C13.1, C14.1
