File: hw/v0p9p5/raspi_connectors.kicad_sch (KiCad schematic)
At the start: 3 parts

Commit message: Updates - candidate board layout
Parts:
- J8: value (none) -> Raspberry_Pi_2_3; footprint (none) -> Connector_PinSocket_2.54mm:PinSocket_2x20_P2.54mm_Vertical
Connections:
- net +3V3 renamed PI_3v3
- net GPIO0: no longer names the net of J8.27 (ID_SD/GPIO0)
- net GPIO1: no longer names the net of J8.28 (ID_SC/GPIO1)
- net GPIO10: no longer names the net of J8.19 (MOSI0/GPIO10)
- net GPIO11: no longer names the net of J8.23 (SCLK0/GPIO11)
- net GPIO12: no longer names the net of J8.32 (PWM0/GPIO12)
- net GPIO13: no longer names the net of J8.33 (PWM1/GPIO13)
- net GPIO14: no longer names the net of J8.8 (GPIO14/TXD)
- net GPIO15: no longer names the net of J8.10 (GPIO15/RXD)
- net GPIO16: no longer names the net of J8.36 (GPIO16)
- net GPIO17: no longer names the net of J8.11 (GPIO17)
- net GPIO18: no longer names the net of J8.12 (GPIO18/PWM0)
- net GPIO19: no longer names the net of J8.35 (GPIO19/MISO1)
- net GPIO20: no longer names the net of J8.38 (GPIO20/MOSI1)
- net GPIO21: no longer names the net of J8.40 (GPIO21/SCLK1)
- net GPIO22: no longer names the net of J8.15 (GPIO22)
- net GPIO23: no longer names the net of J8.16 (GPIO23)
- net GPIO24: no longer names the net of J8.18 (GPIO24)
- net GPIO25: no longer names the net of J8.22 (GPIO25)
- net GPIO26: no longer names the net of J8.37 (GPIO26)
- net GPIO27: no longer names the net of J8.13 (GPIO27)
- net GPIO4: no longer names the net of J8.7 (GCLK0/GPIO4)
- net GPIO5: no longer names the net of J8.29 (GCLK1/GPIO5)
- net GPIO6: no longer names the net of J8.31 (GCLK2/GPIO6)
- net GPIO7: no longer names the net of J8.26 (~{CE1}/GPIO7)
- net GPIO8: no longer names the net of J8.24 (~{CE0}/GPIO8)
- net GPIO9: no longer names the net of J8.21 (MISO0/GPIO9)
- no-connect marks 0 -> 26
