File: hw/v1p1/ras_pi_supercap_ups.kicad_pcb (KiCad board)
At the start: 2 copper layers, 65 x 56 mm, 91 parts, among them J1 Conn_01x03, J2 Conn_01x05, J3 Conn_01x03, J4 Barrel_Jack, J5 171826-4, J6 LEDs and Buttons, J7 STLinkV2 Connector, J8 Raspberry_Pi_2_3, SW1 Reset, U1 KA431SMFTF, U2 KA431SMFTF, U3 KA431SMFTF, U4 KA431SMFTF, U5 KA431SMFTF, U6 AMS1117-3.3, U7 STM8S003F3P, U8 TPS54331DR

Commit message: fix D1 and D7 part number
Parts:
- C20, C22: value 33u -> 47u
Changed lines of the file:
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@@
   (net 28 "Net-(U8-SS)")
   (net 29 "Net-(U8-COMP)")
-  (net 30 "Net-(D1-A1)")
+  (net 30 "Net-(#FLG01-pwr)")
   (net 31 "Net-(D3-A)")
   (net 32 "+12V")
@@
   (net 41 "unconnected-(J8-GPIO15{slash}RXD-Pad10)")
   (net 42 "unconnected-(J8-GPIO17-Pad11)")
-  (net 43 "Net-(D9-K)")
+  (net 43 "Net-(#FLG03-pwr)")
   (net 44 "unconnected-(J8-GPIO18{slash}PWM0-Pad12)")
   (net 45 "unconnected-(J8-GPIO27-Pad13)")
@@
     (tags "SOD-323")
     (property "DigikeyPN" "")
-    (property "LCSC" "C2990493")
+    (property "LCSC" "C312234")
     (property "Sheetfile" "ras_pi_supercap_ups.kicad_sch")
     (property "Sheetname" "")
@@
       (stroke (width 0.1) (type solid)) (layer "F.Fab"))
     (pad "1" smd roundrect (at -1.05 0 270) (size 0.6 0.45) (layers "F.Cu" "F.Paste" "F.Mask") (roundrect_rratio 0.25)
-      (net 30 "Net-(D1-A1)") (pinfunction "A1") (pintype "passive"))
+      (net 30 "Net-(#FLG01-pwr)") (pinfunction "A1") (pintype "passive"))
     (pad "2" smd roundrect (at 1.05 0 270) (size 0.6 0.45) (layers "F.Cu" "F.Paste" "F.Mask") (roundrect_rratio 0.25)
       (net 2 "GND") (pinfunction "A2") (pintype "passive"))
@@
     (tags "SOD-323")
     (property "DigikeyPN" "")
-    (property "LCSC" "C2990493")
+    (property "LCSC" "C312234")
     (property "Sheetfile" "ras_pi_supercap_ups.kicad_sch")
     (property "Sheetname" "")
@@
       (stroke (width 0.1) (type solid)) (layer "F.Fab"))
     (pad "1" smd roundrect (at -0.9125 0 270) (size 1.025 1.4) (layers "F.Cu" "F.Paste" "F.Mask") (roundrect_rratio 0.243902439)
-      (net 30 "Net-(D1-A1)") (pintype "passive"))
+      (net 30 "Net-(#FLG01-pwr)") (pintype "passive"))
     (pad "2" smd roundrect (at 0.9125 0 270) (size 1.025 1.4) (layers "F.Cu" "F.Paste" "F.Mask") (roundrect_rratio 0.243902439)
       (net 7 "VIN_SENSE") (pintype "passive"))
@@
     (descr "Capacitor SMD 0805 (2012 Metric), square (rectangular) end terminal, IPC_7351 nominal, (Body size source: IPC-SM-782 page 76, https://www.pcb-3d.com/wordpress/wp-content/uploads/ipc-sm-782a_amendment_1_and_2.pdf, https://docs.google.com/spreadsheets/d/1BsfQQcO9C6DZCsRaXUlFlo91Tg2WpOkGARC1WS5S8t0/edit?usp=sharing), generated with kicad-footprint-generator")
     (tags "capacitor")
-    (property "LCSC" "C432920")
+    (property "LCSC" "C16780")
     (property "Sheetfile" "12v_buck_converter.kicad_sch")
     (property "Sheetname" "Buck Converter")
@@
         (effects (font (size 0.7 0.7) (thickness 0.1)))
     )
-    (fp_text value "33u" (at 0 1.68 90) (layer "F.Fab")
+    (fp_text value "47u" (at 0 1.68 90) (layer "F.Fab")
         (effects (font (size 1 1) (thickness 0.15)))
     )
@@
     (descr "Capacitor SMD 0805 (2012 Metric), square (rectangular) end terminal, IPC_7351 nominal, (Body size source: IPC-SM-782 page 76, https://www.pcb-3d.com/wordpress/wp-content/uploads/ipc-sm-782a_amendment_1_and_2.pdf, https://docs.google.com/spreadsheets/d/1BsfQQcO9C6DZCsRaXUlFlo91Tg2WpOkGARC1WS5S8t0/edit?usp=sharing), generated with kicad-footprint-generator")
     (tags "capacitor")
-    (property "LCSC" "C432920")
+    (property "LCSC" "C16780")
     (property "Sheetfile" "12v_buck_converter.kicad_sch")
     (property "Sheetname" "Buck Converter")
@@
         (effects (font (size 0.7 0.7) (thickness 0.1)))
     )
-    (fp_text value "33u" (at 0 1.68 90) (layer "F.Fab")
+    (fp_text value "47u" (at 0 1.68 90) (layer "F.Fab")
         (effects (font (size 1 1) (thickness 0.15)))
     )
@@
       (net 1 "VIN") (pintype "passive"))
     (pad "2" smd roundrect (at 1.4 0 90) (size 1.25 1.75) (layers "F.Cu" "F.Paste" "F.Mask") (roundrect_rratio 0.2)
-      (net 30 "Net-(D1-A1)") (pintype "passive"))
+      (net 30 "Net-(#FLG01-pwr)") (pintype "passive"))
     (model "${KICAD6_3DMODEL_DIR}/Fuse.3dshapes/Fuse_1206_3216Metric.wrl"
       (offset (xyz 0 0 0))
@@
       (net 32 "+12V") (pinfunction "K") (pintype "passive"))
     (pad "2" smd roundrect (at 2 0) (size 2.5 1.8) (layers "F.Cu" "F.Paste" "F.Mask") (roundrect_rratio 0.1388888889)
-      (net 30 "Net-(D1-A1)") (pinfunction "A") (pintype "passive"))
+      (net 30 "Net-(#FLG01-pwr)") (pinfunction "A") (pintype "passive"))
     (model "${KICAD6_3DMODEL_DIR}/Diode_SMD.3dshapes/D_SMA.wrl"
       (offset (xyz 0 0 0))
@@
       (stroke (width 0.1) (type solid)) (layer "F.Fab"))
     (pad "1" smd roundrect (at -2 0 270) (size 2.5 1.8) (layers "F.Cu" "F.Paste" "F.Mask") (roundrect_rratio 0.1388888889)
-      (net 43 "Net-(D9-K)") (pinfunction "K") (pintype "passive"))
+      (net 43 "Net-(#FLG03-pwr)") (pinfunction "K") (pintype "passive"))
     (pad "2" smd roundrect (at 2 0 270) (size 2.5 1.8) (layers "F.Cu" "F.Paste" "F.Mask") (roundrect_rratio 0.1388888889)
       (net 6 "+5V") (pinfunction "A") (pintype "passive"))
@@
       ))
     (pad "2" smd custom (at 0.65 0 90) (size 1 0.5) (layers "B.Cu" "B.Mask")
-      (net 43 "Net-(D9-K)") (pinfunction "B") (pintype "passive") (zone_connect 2) (thermal_bridge_angle 45)
+      (net 43 "Net-(#FLG03-pwr)") (pinfunction "B") (pintype "passive") (zone_connect 2) (thermal_bridge_angle 45)
       (options (clearance outline) (anchor rect))
       (primitives
@@
       (net 24 "PI_3v3") (pinfunction "3V3") (pintype "power_in"))
     (pad "2" thru_hole oval locked (at -2.54 0 270) (size 1.7 1.7) (drill 1) (layers "*.Cu" "*.Mask")
-      (net 43 "Net-(D9-K)") (pinfunction "5V") (pintype "power_in"))
+      (net 43 "Net-(#FLG03-pwr)") (pinfunction "5V") (pintype "power_in"))
     (pad "3" thru_hole oval locked (at 0 -2.54 270) (size 1.7 1.7) (drill 1) (layers "*.Cu" "*.Mask")
       (net 4 "I2C_SDA") (pinfunction "SDA/GPIO2") (pintype "bidirectional"))
     (pad "4" thru_hole oval locked (at -2.54 -2.54 270) (size 1.7 1.7) (drill 1) (layers "*.Cu" "*.Mask")
-      (net 43 "Net-(D9-K)") (pinfunction "5V") (pintype "power_in"))
+      (net 43 "Net-(#FLG03-pwr)") (pinfunction "5V") (pintype "power_in"))
     (pad "5" thru_hole oval locked (at 0 -5.08 270) (size 1.7 1.7) (drill 1) (layers "*.Cu" "*.Mask")
       (net 3 "I2C_SCL") (pinfunction "SCL/GPIO3") (pintype "bidirectional"))
