File: hw/v1p1/ras_pi_supercap_ups.kicad_sch (KiCad schematic)
At the start: 66 parts, among them J1 Conn_01x03, J2 Conn_01x05, J3 Conn_01x03, J4 Barrel_Jack, J5 171826-4, J6 LEDs and Buttons, J7 STLinkV2 Connector, SW1 Reset, U1 KA431SMFTF, U2 KA431SMFTF, U3 KA431SMFTF, U4 KA431SMFTF, U5 KA431SMFTF, U6 AMS1117-3.3, U7 STM8S003F3P

Commit message: fix D1 and D7 part number
Parts:
- D1, D7: LCSC C2990493 -> C312234
Changed lines of the file:
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@@
       (effects (font (size 1.27 1.27)) hide)
     )
-    (property "LCSC" "C2990493" (at 41.91 43.18 0)
+    (property "LCSC" "C312234" (at 41.91 43.18 0)
       (effects (font (size 1.27 1.27)) hide)
     )
@@
       (effects (font (size 1.27 1.27)) hide)
     )
-    (property "LCSC" "C2990493" (at 169.164 75.692 0)
-      (effects (font (size 1.27 1.27)) hide)
-    )
+    (property "LCSC" "C312234" (at 169.164 75.692 0)
+      (effects (font (size 1.27 1.27)) hide)
+    )
